File: v0.2/Hardware/LuchtLampje/LuchtLampje.kicad_pcb (KiCad board)
At the start: 2 copper layers, 100 x 100 mm, 19 parts

Commit message: Fixed small typographic issues
Other:
- board text added: "(Different)"
- board text added: "Place NodeMCU with ESP8266 here, with the µUSB to the right -> Assembly instructions and firmware can be found on github.com/pietervdvn/Luchtlichtje Be careful placing leds, they have one flattened side. The flattened side goes in the middle."
- board text added: "Volunteers all over the world run particulate matter sensors. All these sensors send their data to Luftdaten.info, where all this data can be downloaded. This device visualizes data of one such a sensor in real time."
- board text removed: "Different"
- board text removed: "Place NodeMCU with ESP8266 here, with the µUSB to the right -> Assembly instructions and firmware can be found on github.com/pietervdvn/Luchtlichtje Be carefull placing leds, they have one flattened side. The flattened side goes in the middle."
- board text removed: "Volunteers all over the world run particulate matter sensors. All these sensors send their data to Luftdaten.info, where all this data can be downloaded. This device visualises data of one such a sensor in real time."
Changed lines of the file:
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@@
   (layers
     (0 F.Cu signal)
-    (31 B.Cu signal hide)
-    (32 B.Adhes user hide)
-    (33 F.Adhes user hide)
+    (31 B.Cu signal)
+    (32 B.Adhes user)
+    (33 F.Adhes user)
     (34 B.Paste user hide)
-    (35 F.Paste user hide)
+    (35 F.Paste user)
     (36 B.SilkS user hide)
     (37 F.SilkS user)
-    (38 B.Mask user hide)
-    (39 F.Mask user hide)
-    (40 Dwgs.User user hide)
-    (41 Cmts.User user hide)
-    (42 Eco1.User user hide)
-    (43 Eco2.User user hide)
+    (38 B.Mask user)
+    (39 F.Mask user)
+    (40 Dwgs.User user)
+    (41 Cmts.User user)
+    (42 Eco1.User user)
+    (43 Eco2.User user)
     (44 Edge.Cuts user)
-    (45 Margin user hide)
-    (46 B.CrtYd user hide)
-    (47 F.CrtYd user hide)
-    (48 B.Fab user hide)
-    (49 F.Fab user hide)
+    (45 Margin user)
+    (46 B.CrtYd user)
+    (47 F.CrtYd user)
+    (48 B.Fab user)
+    (49 F.Fab user)
   )
   (setup
@@
     )
   )
-  (gr_text Different (at 115.25 135.25) (layer F.SilkS)
+  (gr_text "(Different)" (at 115.25 135.25) (layer F.SilkS)
     (effects (font (size 0.75 0.75) (thickness 0.15)) (justify left))
   )
@@
     (effects (font (size 6 3) (thickness 0.4)) (justify left))
   )
-  (gr_text "WHO year" (at 63.25 85.75) (layer F.Mask)
-    (effects (font (size 3 1.5) (thickness 0.3)) (justify right))
-  )
-  (gr_text "WHO day" (at 63.25 69) (layer F.Mask)
-    (effects (font (size 3 1.5) (thickness 0.3)) (justify right))
-  )
-  (gr_text "EU year" (at 63 62.5) (layer F.Mask)
+  (gr_text "WHO year" (at 63.25 86.75) (layer F.Mask)
+    (effects (font (size 3 1.5) (thickness 0.3)) (justify right))
+  )
+  (gr_text "WHO day" (at 63.25 70.5) (layer F.Mask)
+    (effects (font (size 3 1.5) (thickness 0.3)) (justify right))
+  )
+  (gr_text "EU year" (at 63 63.25) (layer F.Mask)
     (effects (font (size 3 1.5) (thickness 0.3)) (justify right))
   )
@@
     (effects (font (size 6 3) (thickness 0.4)) (justify right))
   )
-  (gr_text "WHO year" (at 111.75 85.75) (layer F.Cu)
+  (gr_text "WHO year" (at 111.5 86.75) (layer F.Cu)
     (effects (font (size 3 1.5) (thickness 0.3)) (justify left))
   )
-  (gr_text "EU year" (at 111.75 69.25) (layer F.Cu)
+  (gr_text "EU year" (at 111.75 70.5) (layer F.Cu)
     (effects (font (size 3 1.5) (thickness 0.3)) (justify left))
   )
-  (gr_text "WHO+EU day" (at 111.75 62.5) (layer F.Cu)
+  (gr_text "WHO+EU day" (at 111.75 63.25) (layer F.Cu)
     (effects (font (size 3 1.5) (thickness 0.3)) (justify left))
   )
@@
     (effects (font (size 1.5 1.5) (thickness 0.3)) (justify mirror))
   )
-  (gr_text "Place NodeMCU with ESP8266 here, \nwith the µUSB to the right ->\n\nAssembly instructions and firmware can be found on\ngithub.com/pietervdvn/Luchtlichtje\n\nBe carefull placing leds, they have one flattened side.\nThe flattened side goes in the middle." (at 113 120.5) (layer B.SilkS)
+  (gr_text "Place NodeMCU with ESP8266 here, \nwith the µUSB to the right ->\n\nAssembly instructions and firmware can be found on\ngithub.com/pietervdvn/Luchtlichtje\n\nBe careful placing leds, they have one flattened side.\nThe flattened side goes in the middle." (at 113 120.5) (layer B.SilkS)
     (effects (font (size 1.5 1.5) (thickness 0.3)) (justify left mirror))
   )
@@
   (gr_arc (start 122.5 145) (end 127.5 145) (angle 90) (layer Edge.Cuts) (width 0.15))
   (gr_arc (start 52.5 145) (end 52.5 150) (angle 90) (layer Edge.Cuts) (width 0.15))
-  (gr_text "Made by\nPieter Vander Vennet" (at 84.5 115.25) (layer F.Cu)
-    (effects (font (size 1.5 1) (thickness 0.25)) (justify left))
+  (gr_text "Made by\nPieter Vander Vennet" (at 84.5 114) (layer F.Cu)
+    (effects (font (size 2.25 2) (thickness 0.5)) (justify left))
   )
   (gr_text "All given values are in µg/m3.\nIf one led is on, the measured value\nis within the range printed next to it.\nIf two leds are on, the measurement is \nwithin the range indicated by the lines.\n\nThe WHO recommends a maximum yearly\naverage of 10µg/m3 of PM2.5; \nthis is indicated with \"WHO Year\". \nThe WHO-recommended day average is \n25µg/m3, indicated similarly.\nOther norms from the EU are indicated\nsimilarly." (at 125.5 74.25) (layer B.SilkS)
     (effects (font (size 1.5 1) (thickness 0.25)) (justify left mirror))
   )
-  (gr_text "Volunteers all over the world run particulate matter sensors.\nAll these sensors send their data to Luftdaten.info,\nwhere all this data can be downloaded.\nThis device visualises data of one such a sensor in real time." (at 52.5 124.75) (layer F.SilkS)
+  (gr_text "Volunteers all over the world run particulate matter sensors.\nAll these sensors send their data to Luftdaten.info,\nwhere all this data can be downloaded.\nThis device visualizes data of one such a sensor in real time." (at 52.5 124.75) (layer F.SilkS)
     (effects (font (size 2 1.5) (thickness 0.3)) (justify left))
   )
@@
   (gr_arc (start 98.75 80) (end 97.5 80) (angle 90) (layer F.SilkS) (width 0.2))
   (gr_line (start 98.75 78.75) (end 99.25 78.75) (layer F.SilkS) (width 0.2))
-  (gr_text "EU year" (at 63 62.5) (layer F.Cu)
-    (effects (font (size 3 1.5) (thickness 0.3)) (justify right))
-  )
-  (gr_text "WHO day" (at 63.25 69) (layer F.Cu)
-    (effects (font (size 3 1.5) (thickness 0.3)) (justify right))
-  )
-  (gr_text "WHO year" (at 63.25 85.75) (layer F.Cu)
+  (gr_text "EU year" (at 63 63.25) (layer F.Cu)
+    (effects (font (size 3 1.5) (thickness 0.3)) (justify right))
+  )
+  (gr_text "WHO day" (at 63.25 70.5) (layer F.Cu)
+    (effects (font (size 3 1.5) (thickness 0.3)) (justify right))
+  )
+  (gr_text "WHO year" (at 63.25 86.75) (layer F.Cu)
     (effects (font (size 3 1.5) (thickness 0.3)) (justify right))
   )
@@
   (gr_arc (start 75 57.5) (end 75 55) (angle 90) (layer F.SilkS) (width 0.2))
   (gr_arc (start 80 57.5) (end 80 60) (angle 90) (layer F.SilkS) (width 0.2))
-  (gr_text "WHO+EU day" (at 111.75 62.5) (layer F.Mask)
+  (gr_text "WHO+EU day" (at 111.75 63.25) (layer F.Mask)
     (effects (font (size 3 1.5) (thickness 0.3)) (justify left))
   )
@@
     (effects (font (size 3 1.5) (thickness 0.3)) (justify left))
   )
-  (gr_text "EU year" (at 111.75 69.25) (layer F.Mask)
+  (gr_text "EU year" (at 111.75 70.5) (layer F.Mask)
     (effects (font (size 3 1.5) (thickness 0.3)) (justify left))
   )
@@
     (effects (font (size 3 1.5) (thickness 0.3)) (justify left))
   )
-  (gr_text "WHO year" (at 111.75 85.75) (layer F.Mask)
+  (gr_text "WHO year" (at 111.5 86.75) (layer F.Mask)
     (effects (font (size 3 1.5) (thickness 0.3)) (justify left))
   )

Commit message: Fixed small typographic issues
Other:
- board text added: "v2018-09-17"
- board text removed: "v2018-08-24"
Changed lines of the file:
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@@
     (34 B.Paste user hide)
     (35 F.Paste user)
-    (36 B.SilkS user hide)
-    (37 F.SilkS user)
+    (36 B.SilkS user)
+    (37 F.SilkS user hide)
     (38 B.Mask user)
     (39 F.Mask user)
@@
   (gr_line (start 147.5 84.75) (end 142.5 82.25) (layer Edge.Cuts) (width 0.15))
   (gr_line (start 142.5 83.25) (end 142.5 82.25) (layer Edge.Cuts) (width 0.15))
-  (gr_text v2018-08-24 (at 121.5 120.5 270) (layer B.SilkS)
+  (gr_text v2018-09-17 (at 121.5 120.5 270) (layer B.SilkS)
     (effects (font (size 1.5 1.5) (thickness 0.3)) (justify mirror))
   )

Commit message: Update firmware
Other:
- net class Default removed

Commit message: Small changes
Other:
- board text added: "How to read? All given values are in µg/m³. If one led is on in a single column, the measured value is within the range printed next to it. If two leds are on, follow both lines to get the range in which the measurment is. The WHO recommends a maximum yearly average of 10µg/m³ of PM2.5; this is indicated with {dblquote}WHO Year{dblquote}. The WHO-recommended maximal daily average is 25µg/m³, indi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"
- board text added: "You can build your own sensor by following the manual on https://sensor.community Many Hackerspaces, Civics Labs, Fablabs and Makerspaces in your area might be running projects too! Get int touch with your community and strive for better air quality together."
- board text added: "v2025-01-04"
- board text removed: "All given values are in µg/m3. If one led is on, the measured value is within the range printed next to it. If two leds are on, the measurement is within the range indicated by the lines. The WHO recommends a maximum yearly average of 10µg/m3 of PM2.5; this is indicated with "WHO Year". The WHO-recommended day average is 25µg/m3, indicated similarly. Other norms from the EU are indicated similarl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"
- board text removed: "You can build your own sensor by following the manual on luftdaten.info Many Hackerspaces, Civics Labs, Fablabs and Makerspaces in your area might be running projects too! Get int touch with your community and strive for better air quality together."
- board text removed: "v2018-09-17"
Changed lines of the file:
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@@
     (effects (font (size 2.25 2) (thickness 0.5)) (justify left))
   )
-  (gr_text "You can build your own sensor by\nfollowing the manual on luftdaten.info\n\nMany Hackerspaces, Civics Labs,\nFablabs and Makerspaces in\nyour area might be running projects too!\nGet int touch with your community\nand strive for better air quality together." (at 80.75 74.25) (layer "B.SilkS")
+  (gr_text "You can build your own sensor by\nfollowing the manual on https://sensor.community\n\nMany Hackerspaces, Civics Labs,\nFablabs and Makerspaces in\nyour area might be running projects too!\nGet int touch with your community\nand strive for better air quality together." (at 80.75 74.25) (layer "B.SilkS")
     (effects (font (size 1.5 1) (thickness 0.25)) (justify left mirror))
   )
@@
     (effects (font (size 1.5 1.5) (thickness 0.3)) (justify mirror))
   )
-  (gr_text "All given values are in µg/m3.\nIf one led is on, the measured value\nis within the range printed next to it.\nIf two leds are on, the measurement is \nwithin the range indicated by the lines.\n\nThe WHO recommends a maximum yearly\naverage of 10µg/m3 of PM2.5; \nthis is indicated with \"WHO Year\". \nThe WHO-recommended day average is \n25µg/m3, indicated similarly.\nOther norms from the EU are indicated\nsimilarly." (at 125.5 74.25) (layer "B.SilkS")
+  (gr_text "How to read?\nAll given values are in µg/m³.\nIf one led is on in a single column, the measured value\nis within the range printed next to it.\nIf two leds are on, follow both lines to get the range in which the measurment is.\n\nThe WHO recommends a maximum yearly\naverage of 10µg/m³ of PM2.5; \nthis is indicated with {dblquote}WHO Year{dblquote}. \nThe WHO-recommended maximal daily average is \n25µg/m³, indicated similarly.\nOther norms from the EU are indicated\nsimilarly." (at 125.5 74.25) (layer "B.SilkS")
     (effects (font (size 1.5 1) (thickness 0.25)) (justify left mirror))
   )
@@
     (effects (font (size 0.75 0.75) (thickness 0.125)) (justify mirror))
   )
-  (gr_text "v2018-09-17" (at 121.5 120.5 270) (layer "B.SilkS")
+  (gr_text "v2025-01-04" (at 121.5 120.5 270) (layer "B.SilkS")
     (effects (font (size 1.5 1.5) (thickness 0.3)) (justify mirror))
   )
